File: Espress0.brd (EAGLE design)
At the start: 36.8 x 39.4 mm, 40 parts, among them CN1 4U#20329, Q2 reset, U1 AP2112K-3.3, U2 2MB Flash, U3 MCP73831T-2ACI/OT

Commit message: Add files via upload
Routing:
- net 3.3V: track 110.5 -> 113.9 mm
- net GND: vias 16 -> 18
Changed lines of the file:
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@@
 </element>
 <element name="C8" library="microbuilder" package="0805-NO" value="10uF" x="9.906" y="25.146" smashed="yes" rot="R90">
-<attribute name="NAME" x="11.811" y="25.4" size="0.8128" layer="121" ratio="18" rot="R90"/>
-<attribute name="VALUE" x="12.446" y="25.273" size="0.4064" layer="121" ratio="10" rot="R90"/>
+<attribute name="NAME" x="11.684" y="25.781" size="0.6096" layer="121" ratio="18" rot="R90"/>
+<attribute name="VALUE" x="12.446" y="25.4" size="0.4064" layer="121" ratio="10" rot="R90"/>
 </element>
 <element name="CN1" library="microbuilder" package="4UCONN_20329_V2" value="4U#20329" x="19.05" y="4.318"/>
@@
 <via x="26.797" y="26.924" extent="1-16" drill="0.35"/>
 <wire x1="18.665" y1="20.705" x2="18.161" y2="21.209" width="0.3048" layer="1"/>
+<via x="7.874" y="20.701" extent="1-16" drill="0.35"/>
+<via x="11.43" y="25.019" extent="1-16" drill="0.35"/>
 <via x="7.493" y="26.924" extent="1-16" drill="0.35"/>
 </signal>
@@
 <wire x1="26.1589" y1="16.168" x2="26.2589" y2="16.068" width="0.4064" layer="1"/>
 <via x="10.922" y="18.288" extent="1-16" drill="0.35"/>
-<wire x1="8.5372" y1="21.66705" x2="8.5372" y2="22.27495" width="0.4064" layer="1"/>
-<wire x1="10.922" y1="19.28225" x2="10.922" y2="18.288" width="0.4064" layer="1"/>
-<wire x1="10.922" y1="19.28225" x2="8.5372" y2="21.66705" width="0.4064" layer="1"/>
 <wire x1="10.922" y1="18.288" x2="8.763" y2="18.288" width="0.4064" layer="1"/>
 <wire x1="6.77" y1="16.295" x2="6.77" y2="15.24" width="0.4064" layer="1"/>
@@
 <wire x1="6.77" y1="16.295" x2="4.015" y2="19.05" width="0.3048" layer="1"/>
 <wire x1="4.015" y1="19.05" x2="2.54" y2="19.05" width="0.3048" layer="1"/>
-<wire x1="9.906" y1="24.196" x2="9.906" y2="23.64375" width="0.4064" layer="1"/>
-<wire x1="9.906" y1="23.64375" x2="9.006125" y2="22.743875" width="0.4064" layer="1"/>
-<wire x1="9.006125" y1="22.743875" x2="8.5372" y2="22.27495" width="0.4064" layer="1"/>
 <wire x1="6.77" y1="15.24" x2="5.08" y2="13.55" width="0.3048" layer="1"/>
 <wire x1="5.08" y1="10.033" x2="5.588" y2="9.525" width="0.3048" layer="1"/>
@@
 <wire x1="24.384" y1="16.168" x2="24.384" y2="14.986" width="0.3048" layer="1"/>
 <wire x1="24.384" y1="14.986" x2="23.749" y2="14.351" width="0.3048" layer="1"/>
-<wire x1="9.006125" y1="22.743875" x2="4.307125" y2="22.743875" width="0.3048" layer="1"/>
-<wire x1="4.307125" y1="22.743875" x2="2.54" y2="24.511" width="0.3048" layer="1"/>
 <wire x1="14.859" y1="14.351" x2="10.922" y2="18.288" width="0.254" layer="16"/>
 <wire x1="17.4173875" y1="15.8976" x2="16.8726125" y2="15.8976" width="0.254" layer="16"/>
@@
 <wire x1="23.749" y1="14.351" x2="18.9639875" y2="14.351" width="0.254" layer="16"/>
 <wire x1="18.9639875" y1="14.351" x2="17.4173875" y2="15.8976" width="0.254" layer="16"/>
+<wire x1="2.54" y1="24.511" x2="2.855" y2="24.196" width="0.4064" layer="1"/>
+<wire x1="2.855" y1="24.196" x2="9.906" y2="24.196" width="0.4064" layer="1"/>
+<wire x1="9.906" y1="24.196" x2="6.731" y2="21.021" width="0.4064" layer="1"/>
+<wire x1="6.731" y1="21.021" x2="6.731" y2="19.685" width="0.4064" layer="1"/>
+<wire x1="6.731" y1="19.685" x2="8.128" y2="18.288" width="0.4064" layer="1"/>
+<wire x1="8.128" y1="18.288" x2="10.922" y2="18.288" width="0.4064" layer="1"/>
 </signal>
 <signal name="N$3">
@@
 <wire x1="16.59399375" y1="23.45199375" x2="13.4803875" y2="26.5656" width="0.254" layer="16"/>
 <wire x1="12.9356125" y1="26.5656" x2="12.1694" y2="25.7993875" width="0.254" layer="16"/>
-<wire x1="9.0452" y1="18.4841875" x2="9.0452" y2="15.9032" width="0.254" layer="16"/>
-<wire x1="12.1694" y1="21.6083875" x2="9.0452" y2="18.4841875" width="0.254" layer="16"/>
 <wire x1="12.1694" y1="25.7993875" x2="12.1694" y2="21.6083875" width="0.254" layer="16"/>
+<wire x1="11.5344" y1="20.9733875" x2="11.5344" y2="20.6540625" width="0.254" layer="16"/>
+<wire x1="12.1694" y1="21.6083875" x2="11.5344" y2="20.9733875" width="0.254" layer="16"/>
+<wire x1="9.0452" y1="18.1648625" x2="9.0452" y2="15.9032" width="0.254" layer="16"/>
+<wire x1="11.5344" y1="20.6540625" x2="9.0452" y2="18.1648625" width="0.254" layer="16"/>
 </signal>
 <signal name="N$1">

Commit message: Add files via upload
Parts:
- moved C4 1.66 mm to (26.9, 30.1), turned to 180 degrees
Routing:
- net VBAT: track 45.9 -> 40.7 mm
- net D3_A3_PA07_RXD_SCK: track 29.2 -> 26.8 mm, vias 2 -> 1
- net VBUS: track 69.3 -> 67.0 mm
- net PA16D_FLASHMOSI: track 12.4 -> 11.6 mm
- net GND: vias 18 -> 19
- net D4_A2_PA06_TXD_MOSI: vias 2 -> 1

Commit message: Add files via upload
Parts:
- added JTAG: (no value), microbuilder:1X02_ROUND
Connections:
- removed net N$3: ATSAMD21E.31, SWC.TP
- removed net N$4: ATSAMD21E.32, SWD.TP
- new net SWC: ATSAMD21E.31, JTAG.2, SWC.TP
- new net SWD: ATSAMD21E.32, JTAG.1, SWD.TP
Routing:
- net SWC: track 0.00 -> 50.2 mm, vias 0 -> 1
- net SWD: track 0.00 -> 24.0 mm, vias 0 -> 2
- net N$3: track 8.34 -> 0.00 mm, vias 1 -> 0
- net N$4: track 5.81 -> 0.00 mm, vias 1 -> 0
- net VBAT: track 40.7 -> 40.2 mm
- net GND: vias 19 -> 21
Other:
- board text added: "SWC"
- board text added: "SWD"

Commit message: Add files via upload
Routing:
- net VBUS: track 67.0 -> 68.6 mm
Changed lines of the file:
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@@
 <element name="CHG" library="microbuilder" package="CHIPLED_0805_NOOUTLINE" value="ORANGE" x="30.353" y="27.686" smashed="yes" rot="R180">
 <attribute name="NAME" x="29.337" y="26.035" size="0.6096" layer="121" ratio="18" rot="R90"/>
-<attribute name="VALUE" x="32.385" y="27.94" size="0.4064" layer="121" ratio="10" rot="R270"/>
+<attribute name="VALUE" x="31.369" y="30.48" size="0.4064" layer="121" ratio="10" rot="R270"/>
 </element>
 <element name="R2" library="microbuilder" package="0603-NO" value="1K" x="30.353" y="23.876" smashed="yes" rot="R270">
@@
 </element>
 <element name="C4" library="microbuilder" package="0805-NO" value="10µF" x="26.924" y="30.099" smashed="yes" rot="R180">
-<attribute name="NAME" x="26.543" y="31.623" size="0.6096" layer="121" ratio="18" rot="R180"/>
-<attribute name="VALUE" x="28.194" y="31.496" size="0.4064" layer="121" ratio="10" rot="R180"/>
+<attribute name="NAME" x="26.035" y="31.877" size="0.6096" layer="121" ratio="18" rot="R180"/>
+<attribute name="VALUE" x="28.575" y="31.75" size="0.4064" layer="121" ratio="10" rot="R180"/>
 </element>
 <element name="R8" library="microbuilder" package="0603-NO" value="10K\" x="23.114" y="26.162" smashed="yes" rot="R90">
@@
 <contactref element="CN1" pad="VBUS"/>
 <via x="21.844" y="6.985" extent="1-16" drill="0.35"/>
-<wire x1="21.844" y1="6.985" x2="25.146" y2="10.922" width="0.4064" layer="1"/>
 <wire x1="25.146" y1="10.922" x2="25.1595" y2="10.922" width="0.4064" layer="1"/>
 <via x="16.383" y="6.985" extent="1-16" drill="0.35"/>
@@
 <wire x1="30.353" y1="28.736" x2="30.353" y2="29.845" width="0.3048" layer="1"/>
 <wire x1="30.353" y1="29.845" x2="30.607" y2="30.099" width="0.3048" layer="1"/>
+<wire x1="21.844" y1="6.985" x2="24.384" y2="6.985" width="0.4064" layer="1"/>
+<wire x1="25.146" y1="7.747" x2="25.146" y2="10.922" width="0.4064" layer="1"/>
+<wire x1="24.384" y1="6.985" x2="25.146" y2="7.747" width="0.4064" layer="1"/>
 </signal>
 <signal name="N$6">
