File: Espress0.sch (EAGLE design)
At the start: 40 parts, among them CN1 4U#20329, Q2 reset, U1 AP2112K-3.3, U2 2MB Flash, U3 MCP73831T-2ACI/OT

Commit message: v0.3
* Layout adjusted and schematic updated, pin header arrangement no longer matches 1:1 with a Trinket m0 board
* Trace diameter for power lines adjusted for 20mm, data for 15mm
* Removed "antennas", trapped copper that is grounded
* Issues re: "Crosstalk" lines were adjusted to have more space and or GND between lines.
Parts:
- added JTAG: (no value), microbuilder:HEADER-1X2ROUND
- JP4: device microbuilder:HEADER-1X576MIL -> adafruit:PINHD-1X1CB
Connections:
- removed net N$3: ATSAMD21E.PA30/I10/SECOM1.2/SWCLK, SWC.TP
- removed net N$4: ATSAMD21E.PA31/I11/SECOM1.3/SWDIO, SWD.TP
- new net SWC: ATSAMD21E.PA30/I10/SECOM1.2/SWCLK, JTAG.2, SWC.TP
- new net SWD: ATSAMD21E.PA31/I11/SECOM1.3/SWDIO, JTAG.1, SWD.TP
- net !RESET: now also JP3.1; no longer JP3.5
- net 3.3V: now also JP3.3; no longer JP1.4, JP4.1
- net D0_A4_PA08_SDA: no longer JP4.4
- net D1_A0_PA02: now also JP4.1; no longer JP4.3
- net D2_A1_PA09_SCL_MISO: no longer JP4.2
- net D3_A3_PA07_RXD_SCK: now also JP1.5; no longer JP3.4
- net D4_A2_PA06_TXD_MOSI: now also JP1.4; no longer JP3.3
- net GND: no longer JP1.5
- net VBAT: now also JP3.4; no longer JP3.1
- net VBUS: now also JP3.5; no longer JP4.5
Other:
- moved on the sheet: JP2

Commit message: v0.5
* New form factor, pins broken out as pads
* 6V/500mA polyfuse between USB 5V+ and the voltage regulator
Parts:
- removed CN1: 4U#20329, microbuilder:USB_MICRO_20329_V2
- removed JP4: (no value), adafruit:PINHD-1X1CB
- removed PA14, PA15, PA18, PA22, PA23, PA27, PA28: TPB1,27, testpad:TPB1,27
- added ALT: (no value), adafruit:PINHD-1X3CB
- added F1: 6V/0.5A, SparkFun-Fuses:PPTC_HALF-AMP
- added LEFT: (no value), microbuilder:HEADER-1X576MIL
- added USB-CONNECTOR: USB-CONNECTOR, SparkFun-Connectors:USB_MICRO-B_FEMALE-SMT
- PWR: value green -> g
- STATUS: value red -> r
- renumbered DOTSTAR to DOTSTAR-A3, JP1 to UP, JP2 to I2C, JP3 to RIGHT
Connections:
- net PA14_FLASHCS renamed PA11_FLASHCS
- removed net N$10: ATSAMD21E.PA14/I14/SERCOM2+4.2, PA14.TP
- removed net N$14: ATSAMD21E.PA18/I2/SERCOM1+3.2, PA18.TP
- removed net N$15: ATSAMD21E.PA28/I8, PA28.TP
- removed net N$16: ATSAMD21E.PA27/I15, PA27.TP
- removed net N$5: ATSAMD21E.PA23/I2C/I7/SERCOM3+5.1/SOF, PA23.TP
- removed net N$7: ATSAMD21E.PA22/I2C/I6/SERCOM3+5.0, PA22.TP
- removed net N$9: ATSAMD21E.PA15/I15/SERCOM3+4.3, PA15.TP
- new net PA14: ATSAMD21E.PA14/I14/SERCOM2+4.2, LEFT.2
- new net PA15: ATSAMD21E.PA15/I15/SERCOM3+4.3, LEFT.3
- new net PA18: ATSAMD21E.PA18/I2/SERCOM1+3.2, LEFT.4
- new net PA22: ALT.2, ATSAMD21E.PA22/I2C/I6/SERCOM3+5.0
- new net PA23: ALT.3, ATSAMD21E.PA23/I2C/I7/SERCOM3+5.1/SOF
- new net PA27: ATSAMD21E.PA27/I15, LEFT.5
- new net PA28: ALT.1, ATSAMD21E.PA28/I8
- new net VBUSRAW: CHG.A, F1.1, RIGHT.5, U3.VDD, USB-CONNECTOR.VBUS
- net D+: now also USB-CONNECTOR.D+; no longer CN1.D+
- net D-: now also USB-CONNECTOR.D-; no longer CN1.D-
- net D1_A0_PA02: now also LEFT.1; no longer JP4.1
- net GND: now also USB-CONNECTOR.GND; no longer CN1.GND
- net VBUS: now also F1.2; no longer CHG.A, CN1.VBUS, RIGHT.5, U3.VDD
